File: hardware/didaktik-gama/didaktik_gama.kicad_sch (KiCad schematic)
At the start: 203 parts, among them J1 Klávesnice, J2 MG, J3 TV, J4 Porty 8255, J5 Napájení 9–12V DC, J6 Video (cinch), SW1 RESET, T1 KSY72, T2 KSY72, T3 KC507, T4 KC507 (BC547), T5 KC507 (Sp TR1 ZTX313), T6 KC507 (Sp TR2 ZTX313), T7 KF517 (Sp TR5 ZTX213), T8 KD139 (Sp TR4 ZTX651/TIP31), U1 UA880D (Z80), U10 4164, U11 4164, U12 4164, U13 4164, U14 4164, U15 4164, U16 4164, U17 2118, U18 2118, U19 2118, U2 27128 (16K EPROM), U20 2118, U21 2118, U22 2118, U23 2118, U24 2118, U25 74LS04, U26 74LS04, U27 74LS00, U28 74LS10, U29 74LS32, U3 8255 (MHB8255), U30 LM1889N, U31 VF modulátor (UM1233 nebo ekv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, U32 MA7805, U4 ULA, U5 74LS157, U6 74LS157, U7 74LS157, U8 74LS157, U9 4164, Y1 14MHz, Y2 4.433619MHz (Sp X2)

Commit message: Replace Spectrum self-oscillating converter with MC34063A boost
MC34063A 9V->12V boost with standard 100uH inductor and Schottky diode
(no custom 1703 coil needed). Upgrade input diode to 1N5822 Schottky and
5V regulator to a pin-compatible switching module (R-78E5.0-1.0).

Co-Authored-By: Claude Opus 5.5 <noreply@anthropic.com>
Claude-Session: https://claude.ai/code/session_01LAVM7Gq9EYiUXiCEdy9ZRx
Parts:
- removed C80: 4u7/16V (úprava dle manuálu), Capacitor_THT:CP_Radial_D5.0mm_P2.00mm, symbol gama:CP
- removed L1: Cívka SPECTRUM 1703, symbol gama:COIL1703
- removed T7: KF517 (Sp TR5 ZTX213), Package_TO_SOT_THT:TO-39-3, symbol gama:PNP
- removed T8: KD139 (Sp TR4 ZTX651/TIP31), Package_TO_SOT_THT:TO-126-3_Vertical, symbol gama:NPN_ECB
- added R71: 0R33 / 0,5 W (Rsc), Resistor_THT:R_Axial_DIN0207_L6.3mm_D2.5mm_P10.16mm_Horizontal, symbol gama:R
- added R74: 1k5 1%, Resistor_THT:R_Axial_DIN0207_L6.3mm_D2.5mm_P10.16mm_Horizontal, symbol gama:R
- added U33: MC34063A, Package_DIP:DIP-8_W7.62mm, symbol gama:MC34063
- C76: value 100n (Sp C43) -> 1n5
- C77: value 47n (Sp C49) -> 100n
- C78: value 100u/16V (Sp C44) -> 330u/25V low ESR; footprint Capacitor_THT:CP_Radial_D6.3mm_P2.50mm -> Capacitor_THT:CP_Radial_D8.0mm_P3.50mm
- C80: renamed from R71; value 1K8 2% (Sp R59) -> 100u/25V; footprint Resistor_THT:R_Axial_DIN0207_L6.3mm_D2.5mm_P10.16mm_Horizontal -> Capacitor_THT:CP_Radial_D6.3mm_P2.50mm; symbol gama:R -> gama:CP
- D12: value KY132/80 (1N4007) -> 1N5822 (Schottky 3A); footprint Diode_THT:D_DO-41_SOD81_P10.16mm_Horizontal -> Diode_THT:D_DO-201AD_P15.24mm_Horizontal
- D14: value BA157 (Sp D15) -> 1N5819 (Schottky)
- L1: renamed from R74; value 15R (Sp R62) -> 100u / 1 A; footprint Resistor_THT:R_Axial_DIN0207_L6.3mm_D2.5mm_P10.16mm_Horizontal -> Inductor_THT:L_Radial_D8.7mm_P5.00mm_Fastron_07HCP; symbol gama:R -> gama:L
- R72: value 1K 2% (Sp R58) -> 180R
- R73: value 270R (Sp R60, Issue 3) -> 13k 1%
- U32: value MA7805 -> R-78E5.0-1.0 (spínaný, náhrada 7805); footprint Package_TO_SOT_THT:TO-220-3_Vertical -> Converter_DCDC:Converter_DCDC_RECOM_R-78E-0.5_THT
Connections:
- net CONV_T7C is gone; now on net +12V: R73.1
- net +12V: now also C77.1; no longer C80.1
- net GND: now also C80.2, R74.2, U33.2 (SWE), U33.4 (GND); no longer R72.2
- net VIN: now also C80.1, R71.1, U33.6 (VCC)
- removed net CONV_DRV: C76.1, L1.1, R73.2
- net CONV_FA renamed BST_SW
- net BST_SW: now also D14.2, U33.1 (SWC)
- net CONV_FB renamed BST_DRV
- net BST_DRV: now also U33.8 (DRV); no longer C80.2
- removed net CONV_SW: C77.1, D14.2
- new net BST_CT: C76.1, U33.3 (CT)
- new net BST_FB: R73.2, R74.1, U33.5 (FB)
- new net BST_IPK: L1.1, R71.2, R72.2, U33.7 (IPK)
Other:
- note added: "MĚNIČ +12 V pro kodér (MC34063A, náhrada měniče ze Spectra)"
- note added: "• U32 spínaný stabilizátor: R-78E5.0-1.0 místo MA7805 (stejné vývody IN-GND-OUT) – Méně tepla (účinnost ~90 %); při rušení obrazu lze vrátit MA7805 na chladiči"
- note added: "• U33 MC34063A (měnič +12 V): náhrada měniče Spectra (TR4/TR5 + cívka 1703) – Zapojení boost podle aplikační poznámky MC34063; Rsc 0R33 = proudové omezení ~0,9 A, Ct 1n5 ~ 30 kHz – ověřit s datasheetem"
- note removed: "MĚNIČ +12 V pro kodér (podle ZX Spectra, TR4/TR5 + cívka 1703)"
- note removed: "• C80, R73: úprava stability měniče z manuálu (4u7 E–B T5, R60 270R) – Doporučeno servisním manuálem Spectra pro desky Issue 2/3"
- note removed: "• L1 (cívka 1703): dvě vinutí: primár VIN–spínač, zpětná vazba R74–báze T8 – Počet závitů / indukčnost cívky Sinclair 1703 schéma neuvádí; začátky vinutí (tečky) dle schématu Spectra"
- note removed: "• T7 KF517: náhrada ZTX213 ověřena katalogovým listem TESLA – PNP, -Uceo 30 V, -Ic 600 mA, Pc 0,8 W, pouzdro K505 (TO-39): vývody E-B-C, výstupek u E; kolektor je spojen s pouzdrem – nesmí se dotýkat okolí"
- note removed: "• T8 KD139: náhrada ZTX651 ověřena katalogovým listem TESLA – NPN, Uceo 80–100 V, Ic 1,5 A (špička 2 A), Ptot 1 W / 12,5 W s chladičem; TO-126 vývody E-C-B (pady 1-2-3), kovová plocha = kolektor – při montáži na chladič izolovat"
- moved on the sheet: L1

Commit message: Replace RF modulator with VGA (RGB 15 kHz) output
YUV->RGB matrix on two AD8032 with black-level and gain trimmers,
LM1881 sync separator with buffered CSYNC/VSYNC via spare 7404 gates,
DE-15 connector. Composite RCA output kept.

Co-Authored-By: Claude Opus 5.5 <noreply@anthropic.com>
Claude-Session: https://claude.ai/code/session_01LAVM7Gq9EYiUXiCEdy9ZRx
Parts:
- removed C10: 100p, Capacitor_THT:C_Disc_D5.0mm_W2.5mm_P5.00mm, symbol gama:C
- removed C63: 100n, Capacitor_THT:C_Disc_D5.0mm_W2.5mm_P5.00mm, symbol gama:C
- removed J3: TV, Connector_Coaxial:BNC_Amphenol_B6252HB-NPP3G-50_Horizontal, symbol gama:CONN_2
- removed U18, U21: 2118, Package_DIP:DIP-16_W7.62mm, symbol gama:2118
- removed unit 6 of U25
- removed unit 5 of U26
- removed unit 2 of U28
- removed U31: VF modulátor (UM1233 nebo ekv.), symbol gama:MODULATOR
- removed U9: 4164, Package_DIP:DIP-16_W7.62mm, symbol gama:4164
- added C24, C30, C41, C81, C82, C83, C84, C85, C86, C87, C88: 100n, Capacitor_THT:C_Disc_D5.0mm_W2.5mm_P5.00mm, symbol gama:C
- added J7: VGA DE-15 (RGB 15 kHz), Connector_Dsub:DSUB-15-HD_Female_Horizontal_P2.29x1.98mm_EdgePinOffset3.03mm_Housed_MountingHolesOffset4.94mm, symbol gama:VGA
- added R100, R82, R89, R97, R99: 75, Resistor_THT:R_Axial_DIN0207_L6.3mm_D2.5mm_P10.16mm_Horizontal, symbol gama:R
- added R20, R45: 470, Resistor_THT:R_Axial_DIN0207_L6.3mm_D2.5mm_P10.16mm_Horizontal, symbol gama:R
- added R27: 330, Resistor_THT:R_Axial_DIN0207_L6.3mm_D2.5mm_P10.16mm_Horizontal, symbol gama:R
- added R76, R77, R79, R83, R84, R86, R90, R94: 1k, Resistor_THT:R_Axial_DIN0207_L6.3mm_D2.5mm_P10.16mm_Horizontal, symbol gama:R
- added R78: 2k2 trimr (kontrast R), Resistor_THT:R_Axial_DIN0207_L6.3mm_D2.5mm_P10.16mm_Horizontal, symbol gama:R
- added R80, R87, R95: 10k, Resistor_THT:R_Axial_DIN0207_L6.3mm_D2.5mm_P10.16mm_Horizontal, symbol gama:R
- added R81: 10k trimr (černá R), Resistor_THT:R_Axial_DIN0207_L6.3mm_D2.5mm_P10.16mm_Horizontal, symbol gama:R
- added R85: 2k2 trimr (kontrast B), Resistor_THT:R_Axial_DIN0207_L6.3mm_D2.5mm_P10.16mm_Horizontal, symbol gama:R
- added R88: 10k trimr (černá B), Resistor_THT:R_Axial_DIN0207_L6.3mm_D2.5mm_P10.16mm_Horizontal, symbol gama:R
- added R91, R92: 2k2, Resistor_THT:R_Axial_DIN0207_L6.3mm_D2.5mm_P10.16mm_Horizontal, symbol gama:R
- added R93: 2k2 trimr (kontrast G), Resistor_THT:R_Axial_DIN0207_L6.3mm_D2.5mm_P10.16mm_Horizontal, symbol gama:R
- added R96: 10k trimr (černá G), Resistor_THT:R_Axial_DIN0207_L6.3mm_D2.5mm_P10.16mm_Horizontal, symbol gama:R
- added R98: 680k, Resistor_THT:R_Axial_DIN0207_L6.3mm_D2.5mm_P10.16mm_Horizontal, symbol gama:R
- added U16: 4164, Package_DIP:DIP-16_W7.62mm, symbol gama:4164
- added unit 3 of U26
- added unit 4 of U26
- added unit 6 of U26
- added unit 2 of U26
- added U34, U35: AD8032AN, Package_DIP:DIP-8_W7.62mm, symbol gama:AD8032
- added U36: LM1881N, Package_DIP:DIP-8_W7.62mm, symbol gama:LM1881
- C10: renamed from C41; value 100n -> 100p
- U18: renamed from R20; value 470 -> 2118; footprint Resistor_THT:R_Axial_DIN0207_L6.3mm_D2.5mm_P10.16mm_Horizontal -> Package_DIP:DIP-16_W7.62mm; symbol gama:R -> gama:2118
- U21: renamed from R27; value 330 -> 2118; footprint Resistor_THT:R_Axial_DIN0207_L6.3mm_D2.5mm_P10.16mm_Horizontal -> Package_DIP:DIP-16_W7.62mm; symbol gama:R -> gama:2118
- U25: renamed from R45; value 470 -> 74LS04; footprint Resistor_THT:R_Axial_DIN0207_L6.3mm_D2.5mm_P10.16mm_Horizontal -> Package_DIP:DIP-14_W7.62mm; symbol gama:R -> gama:7404
- U26: renamed from C24; value 100n -> 74LS04; footprint Capacitor_THT:C_Disc_D5.0mm_W2.5mm_P5.00mm -> Package_DIP:DIP-14_W7.62mm; symbol gama:C -> gama:7404
- U28: renamed from C30; value 100n -> 74LS10; footprint Capacitor_THT:C_Disc_D5.0mm_W2.5mm_P5.00mm -> Package_DIP:DIP-14_W7.62mm; symbol gama:C -> gama:7410
- renumbered U16 to U9
Connections:
- net +5V: now also U18.8 (VCC), U18.9 (VCC), U21.8 (VCC), U21.9 (VCC), C24.1, C30.1, C41.1, C84.1, C85.1, C88.1, R80.1, R87.1, R95.1, U16.8 (VCC), U34.8 (V+), U35.8 (V+), U36.8 (VCC); no longer C10.1, U26.1, U28.1
- net A7_N: now also U28.3
- net BANK: now also U26.11
- net D0: now also U9.14 (Q), U9.2 (D)
- net D1: now also R20.1; no longer U18.1
- net D7: now also U16.14 (Q), U16.2 (D); no longer U9.14 (Q), U9.2 (D)
- net GND: now also U18.16 (GND), U21.16 (GND), C24.2, C30.2, C41.2, C81.2, C82.2, C83.2, C84.2, C85.2, C87.2, C88.2, J7.10 (SYNC_GND), J7.5 (GND), J7.6 (R_GND), J7.7 (G_GND), J7.8 (B_GND), R45.2, R81.2, R88.2, R96.2, R98.2, U16.16 (GND), U34.4 (V-), U35.4 (V-), U35.5 (+INB), U36.4 (GND); no longer U25.2, U26.2, U28.2
- net IORQ_H: now also U28.4
- net LED_K: now also R45.1; no longer U25.1
- net RA0: now also U16.5 (A0)
- net RA1: now also U16.7 (A1)
- net RA2: now also U16.6 (A2)
- net RA3: now also U16.12 (A3)
- net RA4: now also U16.11 (A4)
- net RA5: now also U16.10 (A5)
- net RA6: now also U16.13 (A6)
- net RA7: now also U16.9 (A7)
- net RESET: now also U25.12
- net U: now also R84.1, R91.1
- net V: now also R77.1, R92.1
- net VA0: now also U18.5 (A0), U21.5 (A0), R27.2; no longer U21.2
- net VA1: now also U18.11 (A4), U21.11 (A4)
- net VA2: now also U18.7 (A1), U21.7 (A1)
- net VA3: now also U18.13 (A6), U21.13 (A6)
- net VA4: now also U18.12 (A3), U21.12 (A3)
- net VA5: now also U18.10 (A5), U21.10 (A5)
- net VA6: now also U18.6 (A2), U21.6 (A2)
- net VD1: now also U18.14 (Q), R20.2
- net VD4: now also U21.14 (Q), U21.2 (D)
- net VM0: now also R27.1; no longer U21.1
- net Y: now also C86.1, R76.1, R83.1, R90.1
- net ~{BANKSEL}: now also U26.10
- net ~{CAS64}: now also U16.15 (~{CAS})
- net ~{CS8255}: now also U28.6
- net ~{M1}: now also U28.5
- net ~{MREQ}: now also C10.1
- net ~{RAS64}: now also U16.4 (~{RAS})
- net ~{RESET}: now also U25.13
- net ~{VCAS}: now also U18.15 (~{CAS}), U21.15 (~{CAS})
- net ~{VRAS}: now also U18.4 (~{RAS}), U21.4 (~{RAS})
- net ~{VWE}: now also U18.3 (~{WE}), U21.3 (~{WE})
- net ~{WE64}: now also U16.3 (~{WE})
- new net B_BLK: C82.1, R86.2, R87.2, R88.1
- new net B_FB: R85.2, R86.1, U34.6 (-INB)
- new net B_OUT: R85.1, R89.1, U34.7 (OUTB)
- new net B_SUM: R83.2, R84.2, U34.5 (+INB)
- new net CSYNC_I: U26.4, U26.5
- new net G_BLK: C83.1, R94.2, R95.2, R96.1
- new net G_FB: R91.2, R92.2, R93.2, R94.1, U35.2 (-INA)
- new net G_OUT: R93.1, R97.1, U35.1 (OUTA)
- new net G_Y: R90.2, U35.3 (+INA)
- new net R_BLK: C81.1, R79.2, R80.2, R81.1
- new net R_FB: R78.2, R79.1, U34.2 (-INA)
- new net R_OUT: R78.1, R82.1, U34.1 (OUTA)
- new net R_SUM: R76.2, R77.2, U34.3 (+INA)
- new net SYNC_IN: C86.2, U36.2 (VIDEO_IN)
- new net SYNC_RSET: C87.1, R98.1, U36.6 (RSET)
- new net U35B_OUT: U35.6 (-INB), U35.7 (OUTB)
- new net VGA_B: J7.3 (BLUE), R89.2
- new net VGA_G: J7.2 (GREEN), R97.2
- new net VGA_HS: J7.13 (HSYNC), R99.2
- new net VGA_R: J7.1 (RED), R82.2
- new net VGA_VS: J7.14 (VSYNC), R100.2
- new net VSYNC_I: U26.13, U26.8
- new net ~{CSYNC_B}: R99.1, U26.6
- new net ~{CSYNC}: U26.3, U36.1 (CSYNC)
- new net ~{VSYNC_B}: R100.1, U26.12
- new net ~{VSYNC}: U26.9, U36.3 (VSYNC)
- no-connect marks 6 -> 13
Other:
- note added: "KODÉR PAL LM1889 + KOMPOZITNÍ VÝSTUP"
- note added: "VGA VÝSTUP RGB 15 kHz (matice YUV->RGB + LM1881) – místo modulátoru"
- note added: "• R76–R97 (matice YUV->RGB): poměry R = Y+V, B = Y+U, G = Y-(U+V) – Úrovně U/V z ULA nejsou dokumentované – trimry nastavit podle bílé/černé a barevných pruhů; G kanál nejcitlivější"
- note added: "• U31/J3 modulátor: odstraněn – Nahrazen výstupem VGA; zůstává kompozitní cinch J6"
- note added: "• U36 LM1881: vstup z Y přes 100n, Rset 680k || 100n – Podle katalogového listu LM1881; ověřit, že Y z ULA má 0,5–2 Vpp"
- note added: "• VGA výstup (U34–U36, J7): RGB 15,6 kHz + CSYNC na pinu 13, VSYNC na pinu 14 – Běžný VGA monitor chce 31 kHz – potřeba monitor s 15 kHz nebo převodník (GBS-8200, OSSC, RetroTINK)"
- note removed: "KODÉR PAL LM1889 + VIDEO VÝSTUP"
- note removed: "• U31 (modulátor): vývody modulu +5V / VIDEO / GND / VF – Modul je na předloze jen blok; pořadí vývodů podle konkrétního modulu"
- moved on the sheet: C10, C76, C77, C78, C79, C80, D14, L1, R71, R72, R73, R74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

Commit message: Switch to digital RGB VGA output from a CPLD ULA replacement
ULA socket takes a CPLD module (XC95144XL, zx_ula firmware) that outputs
digital R/G/B/BRIGHT and sync on J8. 74HCT244 drives colours and sync,
74HCT08 gates BRIGHT per colour, resistor DAC into the DE-15 connector.
Removed LM1889 coder, +12V converter, composite output and the analog
YUV->RGB matrix with LM1881.

Co-Authored-By: Claude Opus 5.5 <noreply@anthropic.com>
Claude-Session: https://claude.ai/code/session_01LAVM7Gq9EYiUXiCEdy9ZRx
Parts:
- removed C10: 100p, Capacitor_THT:C_Disc_D5.0mm_W2.5mm_P5.00mm, symbol gama:C
- removed C27, C38, C46, C77, C83, C84, C85, C86, C87, C88: 100n, Capacitor_THT:C_Disc_D5.0mm_W2.5mm_P5.00mm, symbol gama:C
- removed C62: 220u/10V, Capacitor_THT:CP_Radial_D6.3mm_P2.50mm, symbol gama:CP
- removed C64: 47n (Sp C33), Capacitor_THT:C_Disc_D5.0mm_W2.5mm_P5.00mm, symbol gama:C
- removed C65: 22u/16V (Sp C34), Capacitor_THT:CP_Radial_D5.0mm_P2.00mm, symbol gama:CP
- removed C66: 47n (Sp C40), Capacitor_THT:C_Disc_D5.0mm_W2.5mm_P5.00mm, symbol gama:C
- removed C67: trimr (Sp VC2), Capacitor_THT:C_Disc_D5.0mm_W2.5mm_P5.00mm, symbol gama:C
- removed C71: 33p (Sp C38), Capacitor_THT:C_Disc_D5.0mm_W2.5mm_P5.00mm, symbol gama:C
- removed C72: 10n (Sp C39), Capacitor_THT:C_Disc_D5.0mm_W2.5mm_P5.00mm, symbol gama:C
- removed C73: 22u/16V (Sp C65), Capacitor_THT:CP_Radial_D5.0mm_P2.00mm, symbol gama:CP
- removed C74: 47n (Sp C61), Capacitor_THT:C_Disc_D5.0mm_W2.5mm_P5.00mm, symbol gama:C
- removed C75: 22u/16V (Sp C25), Capacitor_THT:CP_Radial_D5.0mm_P2.00mm, symbol gama:CP
- removed C76: 1n5, Capacitor_THT:C_Disc_D5.0mm_W2.5mm_P5.00mm, symbol gama:C
- removed C78: 330u/25V low ESR, Capacitor_THT:CP_Radial_D8.0mm_P3.50mm, symbol gama:CP
- removed C79: 100u/16V (Sp C45), Capacitor_THT:CP_Radial_D6.3mm_P2.50mm, symbol gama:CP
- removed C80: 100u/25V, Capacitor_THT:CP_Radial_D6.3mm_P2.50mm, symbol gama:CP
- removed D14: 1N5819 (Schottky), Diode_THT:D_DO-41_SOD81_P10.16mm_Horizontal, symbol gama:D
- removed J6: Video (cinch), Connector_Coaxial:CONN_RCA_Horizontal, symbol gama:CONN_2
- removed L1: 100u / 1 A, Inductor_THT:L_Radial_D8.7mm_P5.00mm_Fastron_07HCP, symbol gama:L
- removed R100, R47, R97, R99: 75, Resistor_THT:R_Axial_DIN0207_L6.3mm_D2.5mm_P10.16mm_Horizontal, symbol gama:R
- removed R38: 8k2, Resistor_THT:R_Axial_DIN0207_L6.3mm_D2.5mm_P10.16mm_Horizontal, symbol gama:R
- removed R46: 470, Resistor_THT:R_Axial_DIN0207_L6.3mm_D2.5mm_P10.16mm_Horizontal, symbol gama:R
- removed R48: 3K3 (Sp R38), Resistor_THT:R_Axial_DIN0207_L6.3mm_D2.5mm_P10.16mm_Horizontal, symbol gama:R
- removed R49: 2K2 trimr (Sp VR1), Resistor_THT:R_Axial_DIN0207_L6.3mm_D2.5mm_P10.16mm_Horizontal, symbol gama:R
- removed R50: 220R (Sp R56), Resistor_THT:R_Axial_DIN0207_L6.3mm_D2.5mm_P10.16mm_Horizontal, symbol gama:R
- removed R51: 3K3 (Sp R39), Resistor_THT:R_Axial_DIN0207_L6.3mm_D2.5mm_P10.16mm_Horizontal, symbol gama:R
- removed R52: 2K2 trimr (Sp VR2), Resistor_THT:R_Axial_DIN0207_L6.3mm_D2.5mm_P10.16mm_Horizontal, symbol gama:R
- removed R53: 330R (Sp R57), Resistor_THT:R_Axial_DIN0207_L6.3mm_D2.5mm_P10.16mm_Horizontal, symbol gama:R
- removed R54: 1K (Sp R40), Resistor_THT:R_Axial_DIN0207_L6.3mm_D2.5mm_P10.16mm_Horizontal, symbol gama:R
- removed R55: 1K5 (Sp R41), Resistor_THT:R_Axial_DIN0207_L6.3mm_D2.5mm_P10.16mm_Horizontal, symbol gama:R
- removed R56: 1K (Sp R42), Resistor_THT:R_Axial_DIN0207_L6.3mm_D2.5mm_P10.16mm_Horizontal, symbol gama:R
- removed R58: 3K (Sp R43), Resistor_THT:R_Axial_DIN0207_L6.3mm_D2.5mm_P10.16mm_Horizontal, symbol gama:R
- removed R59: 5K1 (Sp R44), Resistor_THT:R_Axial_DIN0207_L6.3mm_D2.5mm_P10.16mm_Horizontal, symbol gama:R
- removed R61: 1K (Sp R46), Resistor_THT:R_Axial_DIN0207_L6.3mm_D2.5mm_P10.16mm_Horizontal, symbol gama:R
- removed R62: 10K (Sp R72), Resistor_THT:R_Axial_DIN0207_L6.3mm_D2.5mm_P10.16mm_Horizontal, symbol gama:R
- removed R65: 4K7 (Sp R50), Resistor_THT:R_Axial_DIN0207_L6.3mm_D2.5mm_P10.16mm_Horizontal, symbol gama:R
- removed R66: 18K (Sp R49), Resistor_THT:R_Axial_DIN0207_L6.3mm_D2.5mm_P10.16mm_Horizontal, symbol gama:R
- removed R67: 2K2 (Sp R52), Resistor_THT:R_Axial_DIN0207_L6.3mm_D2.5mm_P10.16mm_Horizontal, symbol gama:R
- removed R68: 2K2 (Sp R51), Resistor_THT:R_Axial_DIN0207_L6.3mm_D2.5mm_P10.16mm_Horizontal, symbol gama:R
- removed R69: 390R (Sp R53), Resistor_THT:R_Axial_DIN0207_L6.3mm_D2.5mm_P10.16mm_Horizontal, symbol gama:R
- removed R70: 15R (Sp R64), Resistor_THT:R_Axial_DIN0207_L6.3mm_D2.5mm_P10.16mm_Horizontal, symbol gama:R
- removed R71: 0R33 / 0,5 W (Rsc), Resistor_THT:R_Axial_DIN0207_L6.3mm_D2.5mm_P10.16mm_Horizontal, symbol gama:R
- removed R72: 180R, Resistor_THT:R_Axial_DIN0207_L6.3mm_D2.5mm_P10.16mm_Horizontal, symbol gama:R
- removed R73: 13k 1%, Resistor_THT:R_Axial_DIN0207_L6.3mm_D2.5mm_P10.16mm_Horizontal, symbol gama:R
- removed R74: 1k5 1%, Resistor_THT:R_Axial_DIN0207_L6.3mm_D2.5mm_P10.16mm_Horizontal, symbol gama:R
- removed R75: 15R (Sp R61), Resistor_THT:R_Axial_DIN0207_L6.3mm_D2.5mm_P10.16mm_Horizontal, symbol gama:R
- removed R79, R90, R94: 1k, Resistor_THT:R_Axial_DIN0207_L6.3mm_D2.5mm_P10.16mm_Horizontal, symbol gama:R
- removed R80, R87, R95: 10k, Resistor_THT:R_Axial_DIN0207_L6.3mm_D2.5mm_P10.16mm_Horizontal, symbol gama:R
- removed R81: 10k trimr (černá R), Resistor_THT:R_Axial_DIN0207_L6.3mm_D2.5mm_P10.16mm_Horizontal, symbol gama:R
- removed R88: 10k trimr (černá B), Resistor_THT:R_Axial_DIN0207_L6.3mm_D2.5mm_P10.16mm_Horizontal, symbol gama:R
- removed R91, R92: 2k2, Resistor_THT:R_Axial_DIN0207_L6.3mm_D2.5mm_P10.16mm_Horizontal, symbol gama:R
- removed R93: 2k2 trimr (kontrast G), Resistor_THT:R_Axial_DIN0207_L6.3mm_D2.5mm_P10.16mm_Horizontal, symbol gama:R
- removed R96: 10k trimr (černá G), Resistor_THT:R_Axial_DIN0207_L6.3mm_D2.5mm_P10.16mm_Horizontal, symbol gama:R
- removed R98: 680k, Resistor_THT:R_Axial_DIN0207_L6.3mm_D2.5mm_P10.16mm_Horizontal, symbol gama:R
- removed T4: KC507 (BC547), Package_TO_SOT_THT:TO-18-3, symbol gama:NPN
- removed T5: KC507 (Sp TR1 ZTX313), Package_TO_SOT_THT:TO-18-3, symbol gama:NPN
- removed T6: KC507 (Sp TR2 ZTX313), Package_TO_SOT_THT:TO-18-3, symbol gama:NPN
- removed U14: 4164, Package_DIP:DIP-16_W7.62mm, symbol gama:4164
- removed unit 3 of U26
- removed unit 4 of U26
- removed unit 6 of U26
- removed unit 2 of U26
- removed U30: LM1889N, Package_DIP:DIP-18_W7.62mm, symbol gama:LM1889
- removed U33: MC34063A, Package_DIP:DIP-8_W7.62mm, symbol gama:MC34063
- removed U34, U35: AD8032AN, Package_DIP:DIP-8_W7.62mm, symbol gama:AD8032
- removed U36: LM1881N, Package_DIP:DIP-8_W7.62mm, symbol gama:LM1881
- added J8: RGB z modulu ULA, Connector_PinHeader_2.54mm:PinHeader_1x08_P2.54mm_Vertical, symbol gama:CONN_8
- added R24: 470, Resistor_THT:R_Axial_DIN0207_L6.3mm_D2.5mm_P10.16mm_Horizontal, symbol gama:R
- added R32: 330, Resistor_THT:R_Axial_DIN0207_L6.3mm_D2.5mm_P10.16mm_Horizontal, symbol gama:R
- added U11, U16: 4164, Package_DIP:DIP-16_W7.62mm, symbol gama:4164
- added unit 1 of U25
- added unit 5 of U26
- added U37: 74HCT244, Package_DIP:DIP-20_W7.62mm, symbol gama:74HCT244
- added U38: 74HCT08, Package_DIP:DIP-14_W7.62mm, symbol gama:74HCT08
- C10: renamed from U11; value 4164 -> 100p; footprint Package_DIP:DIP-16_W7.62mm -> Capacitor_THT:C_Disc_D5.0mm_W2.5mm_P5.00mm; symbol gama:4164 -> gama:C
- C27: renamed from U16; value 4164 -> 100n; footprint Package_DIP:DIP-16_W7.62mm -> Capacitor_THT:C_Disc_D5.0mm_W2.5mm_P5.00mm; symbol gama:4164 -> gama:C
- C38: renamed from U25; value 74LS04 -> 100n; footprint Package_DIP:DIP-14_W7.62mm -> Capacitor_THT:C_Disc_D5.0mm_W2.5mm_P5.00mm; symbol gama:7404 -> gama:C
- C46: renamed from U26; value 74LS04 -> 100n; footprint Package_DIP:DIP-14_W7.62mm -> Capacitor_THT:C_Disc_D5.0mm_W2.5mm_P5.00mm; symbol gama:7404 -> gama:C
- R38: renamed from R32; value 330 -> 8k2
- R76: value 1k -> 680
- R77: value 1k -> 1k5
- R78: value 2k2 trimr (kontrast R) -> 680
- R79: renamed from Y2; value 4.433619MHz (Sp X2) -> 1k5; footprint Crystal:Crystal_HC49-4H_Vertical -> Resistor_THT:R_Axial_DIN0207_L6.3mm_D2.5mm_P10.16mm_Horizontal; symbol gama:XTAL -> gama:R
- R80: renamed from R60; value 1K (Sp R45) -> 680
- R81: renamed from C68; value 33p (Sp C37) -> 1k5; footprint Capacitor_THT:C_Disc_D5.0mm_W2.5mm_P5.00mm -> Resistor_THT:R_Axial_DIN0207_L6.3mm_D2.5mm_P10.16mm_Horizontal; symbol gama:C -> gama:R
- R83: value 1k -> 75
- R84, R86: value 1k -> 10k
- R85: value 2k2 trimr (kontrast B) -> 10k
- R87: renamed from R63; value 220R (Sp R47) -> 10k
- R88: renamed from R64; value 4K7 (Sp R48) -> 10k
- R89: value 75 -> 10k
- U14: renamed from R24; value 470 -> 4164; footprint Resistor_THT:R_Axial_DIN0207_L6.3mm_D2.5mm_P10.16mm_Horizontal -> Package_DIP:DIP-16_W7.62mm; symbol gama:R -> gama:4164
Connections:
- net R_BLK is gone; now on net +5V: C81.1
- net R_FB is gone; now on net VGA_G: R78.2
- net R_SUM is gone; now on net VGA_R: R76.2, R77.2
- net +5V: now also C27.1, C38.1, C46.1, C82.1, R38.1, R88.1, R89.1, U14.8 (VCC), J8.7, U11.8 (VCC), U16.8 (VCC), U37.20 (VCC), U38.14 (VCC); no longer C10.8 (VCC), C27.8 (VCC)
- net BANK: now also U26.11; no longer C46.11
- net D2: now also U11.14 (Q), U11.2 (D); no longer C10.14 (Q), C10.2 (D)
- net D3: now also R38.2
- net D5: now also U14.14 (Q), U14.2 (D), R24.1; no longer U14.1
- net D7: now also U16.14 (Q), U16.2 (D); no longer C27.14 (Q), C27.2 (D)
- net GND: now also C10.2, C27.2, C38.2, C46.2, R84.2, R85.2, R86.2, U14.16 (GND), J8.8, U11.16 (GND), U16.16 (GND), U37.1 (~{1OE}), U37.10 (GND), U37.13 (2A2), U37.15 (2A3), U37.17 (2A4), U37.19 (~{2OE}), U38.12 (4A), U38.13 (4B), U38.7 (GND); no longer C10.16 (GND), C27.16 (GND), R81.2
- net RA0: now also U14.5 (A0), U11.5 (A0), U16.5 (A0); no longer C10.5 (A0), C27.5 (A0)
- net RA1: now also U14.7 (A1), U11.7 (A1), U16.7 (A1); no longer C10.7 (A1), C27.7 (A1)
- net RA2: now also U14.6 (A2), U11.6 (A2), U16.6 (A2); no longer C10.6 (A2), C27.6 (A2)
- net RA3: now also U14.12 (A3), U11.12 (A3), U16.12 (A3); no longer C10.12 (A3), C27.12 (A3)
- net RA4: now also U14.11 (A4), U11.11 (A4), U16.11 (A4); no longer C10.11 (A4), C27.11 (A4)
- net RA5: now also U14.10 (A5), U11.10 (A5), U16.10 (A5); no longer C10.10 (A5), C27.10 (A5)
- net RA6: now also U14.13 (A6), U11.13 (A6), U16.13 (A6); no longer C10.13 (A6), C27.13 (A6)
- net RA7: now also U14.9 (A7), U11.9 (A7), U16.9 (A7); no longer C10.9 (A7), C27.9 (A7)
- net VA5: now also R32.2; no longer R38.2
- net VD5: now also R24.2; no longer U14.2
- net VGA_B: now also R80.2, R81.2; no longer R89.2
- net VGA_G: now also R79.2
- net VGA_HS: now also R82.2
- net VGA_R: no longer R82.2
- net VGA_VS: now also R83.2
- net VM5: now also R32.1; no longer R38.1
- net WR_I: now also U25.2; no longer C38.2
- net ~{BANKSEL}: now also U26.10; no longer C46.10
- net ~{CAS64}: now also U14.15 (~{CAS}), U11.15 (~{CAS}), U16.15 (~{CAS}); no longer C10.15 (~{CAS}), C27.15 (~{CAS})
- net ~{MREQ}: now also C10.1
- net ~{RAS64}: now also U14.4 (~{RAS}), U11.4 (~{RAS}), U16.4 (~{RAS}); no longer C10.4 (~{RAS}), C27.4 (~{RAS})
- net ~{WE64}: now also U14.3 (~{WE}), U11.3 (~{WE}), U16.3 (~{WE}); no longer C10.3 (~{WE}), C27.3 (~{WE})
- net ~{WR}: now also U25.1; no longer C38.1
- removed net B_BLK: C82.1, R86.2
- net B_FB renamed RGB_B
- net RGB_B: now also J8.3, U37.6 (1A3), U38.9 (3A); no longer R85.2
- net B_OUT renamed RGB_G
- net RGB_G: now also J8.2, U37.4 (1A2), U38.4 (2A); no longer R89.1
- removed net B_SUM: R83.2, R84.2
- net CH_LAG renamed DACB_B
- net DACB_B: now also U38.8 (3Y); no longer R80.2
- net CH_N2 renamed DACB_G
- net DACB_G: now also U38.6 (2Y)
- net CH_N3 renamed DAC_B
- net DAC_B: now also U37.14 (1Y3); no longer R79.2
- net R_OUT renamed DAC_G
- net DAC_G: now also U37.16 (1Y2); no longer R82.1
- net T5_B renamed ~{RGB_CSYNC}
- net ~{RGB_CSYNC}: now also J8.5, U37.8 (1A4)
- net U: no longer names the net of U4.15 (U)
- net U: no longer R84.1
- net V: no longer names the net of U4.16 (V)
- net V: no longer R77.1
- removed net Y: R76.1, R83.1, R87.1, R88.1, U4.17 (Y)
- new net DACB_R: R77.1, U38.3 (1Y)
- new net DAC_R: R76.1, U37.18 (1Y1)
- new net RGB_I: J8.4, R87.1, U38.10 (3B), U38.2 (1B), U38.5 (2B)
- new net RGB_R: J8.1, R84.1, U37.2 (1A1), U38.1 (1A)
- new net VGA_HS_D: R82.1, U37.12 (1Y4)
- new net VGA_VS_D: R83.1, U37.9 (2Y1)
- new net ~{RGB_VSYNC}: J8.6, R89.2, U37.11 (2A1)
- no-connect marks 13 -> 18
Other:
- note added: "VGA VÝSTUP (digitální RGB z modulu ULA s CPLD, 15 kHz)"
- note added: "• J8 / VGA výstup: digitální RGB + BRIGHT + CSYNC/VSYNC z modulu, 15,6 kHz – Běžný VGA monitor chce 31 kHz – potřeba monitor s 15 kHz nebo převodník (GBS-8200, OSSC, RetroTINK)"
- note added: "• R76–R81 (převodník): 680R + 1k5 do 75R monitoru: 0,50 V normální, 0,69 V jas – Vypočteno pro výstup 74HCT244 při 5 V; přesnost závisí na výstupním odporu hradla"
- note added: "• U4 patice ULA: osadit modul s CPLD (XC95144XL + firmware zx_ula, GPL) místo originální ULA – Modul je samostatná deska (40 vývodů do patice + výstup RGB na J8) – zatím nenakreslen; piny 15–17 (U, V, Y) nezapojeny"
- note removed: "KODÉR PAL LM1889 + KOMPOZITNÍ VÝSTUP"
- note removed: "MĚNIČ +12 V pro kodér (MC34063A, náhrada měniče ze Spectra)"
- note removed: "VGA VÝSTUP RGB 15 kHz (matice YUV->RGB + LM1881) – místo modulátoru"
- note removed: "• R76–R97 (matice YUV->RGB): poměry R = Y+V, B = Y+U, G = Y-(U+V) – Úrovně U/V z ULA nejsou dokumentované – trimry nastavit podle bílé/černé a barevných pruhů; G kanál nejcitlivější"
- note removed: "• T4, R46, C62, R47, J6: kompozitní video výstup – Doplněno (na předloze není) – přímý výstup CVBS pro monitor/TV se vstupem AV, obchází modulátor"
- note removed: "• U30 LM1889 + okolí: překresleno ze schématu ZX Spectrum Issue 1/2 – Předloha Gamy má jen blok KÓDER – ověřit, že Gama používá stejné zapojení (typ obvodu na desce)"
- note removed: "• U30 pin 16: chroma supply na +12VA – Ve schématu Spectra není spoj pinu 16 jasně vidět; podle manuálu je to napájení chroma"
- note removed: "• U31/J3 modulátor: odstraněn – Nahrazen výstupem VGA; zůstává kompozitní cinch J6"
- note removed: "• U33 MC34063A (měnič +12 V): náhrada měniče Spectra (TR4/TR5 + cívka 1703) – Zapojení boost podle aplikační poznámky MC34063; Rsc 0R33 = proudové omezení ~0,9 A, Ct 1n5 ~ 30 kHz – ověřit s datasheetem"
- note removed: "• U36 LM1881: vstup z Y přes 100n, Rset 680k || 100n – Podle katalogového listu LM1881; ověřit, že Y z ULA má 0,5–2 Vpp"
- note removed: "• VGA výstup (U34–U36, J7): RGB 15,6 kHz + CSYNC na pinu 13, VSYNC na pinu 14 – Běžný VGA monitor chce 31 kHz – potřeba monitor s 15 kHz nebo převodník (GBS-8200, OSSC, RetroTINK)"
- moved on the sheet: C38, C46, R38, R80, R87, R88
