File: hardware/didaktik-gama/didaktik_gama.kicad_pcb (KiCad board)
At the start: 4 copper layers, 300 x 225 mm, 212 parts, among them J1 Klávesnice, J10 Linkový výstup (jack 3,5 mm), J2 MG, J4 Porty 8255, J5 Napájení 9–12V DC, J7 VGA DE-15 (RGB 15 kHz), J8 RGB + zvuk z modulu ULA, J9 Reproduktor 8 ohm, SW1 RESET, T1 KSY72, T2 KSY72, T3 KC507, U1 UA880D (Z80), U10 4164, U11 4164, U12 4164, U13 4164, U14 4164, U15 4164, U16 4164, U17 2118, U18 2118, U19 2118, U2 27128 (16K EPROM), U20 2118, U21 2118, U22 2118, U23 2118, U24 2118, U25 74LS04, U26 74LS04, U27 74LS00, U28 74LS10, U29 74LS32, U3 8255 (MHB8255), U32 R-78E5.0-1.0 (spínaný, náhrad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, U37 74HCT244, U38 74HCT08, U39 Raspberry Pi Pico (USB host), U4 ULA, U40 74LVC245, U41 74LVC07, U42 YM2149F (nebo AY-3-8910), U43 74HCT11, U44 74HCT74, U45 LM386N-1, U5 74LS157, U6 74LS157, U7 74LS157, U8 74LS157, U9 4164, Y1 14MHz

Commit message: Add ULA CPLD module PCB and keep main board J8 clear of the module
gen_pcb_modul.py builds ula_cpld_modul.kicad_pcb: 70x50 mm 2-layer,
DIP-40 pin field into the ULA socket with courtyards only around the
pin rows, TQFP-100 CPLD above, LDO/oscillator/resistors between the
rows, J2 and JTAG on the sides, GND pour on both layers. Main board J8
moved to the right edge outside the module footprint.

Co-Authored-By: Claude Opus 5.5 <noreply@anthropic.com>
Claude-Session: https://claude.ai/code/session_01LAVM7Gq9EYiUXiCEdy9ZRx
Parts:
- moved D2 270.3 mm to (67.1, 100.3)
- moved J8 26.6 mm to (353.0, 76.6), turned to 0 degrees
- moved D5 11.3 mm to (100.9, 100.3)
- moved D3 11.3 mm to (78.3, 100.3)
- moved D4 11.3 mm to (89.6, 100.3)
- moved D6 11.3 mm to (112.2, 100.3)
- moved D7 11.3 mm to (123.4, 100.3)
- moved D8 11.3 mm to (134.7, 100.3)
